File: Electrical/MotorPowerControl/MotorPowerControl.kicad_pcb (KiCad board)
At the start: 2 copper layers, 10 parts, among them J1 Conn_01x03, J2 178.6164.0002, J3 Conn_01x03, J4 178.6164.0002, J5 178.6164.0002, J6 178.6164.0002

Commit message: Verified Peripheral and Motor power controllers
Parts:
- removed J3: Conn_01x03, Connector_Wire:SolderWirePad_1x03_P7.62mm_Drill2.5mm
- added H2: MountingHole, MountingHole:MountingHole_3.2mm_M3, F.Cu at (169.0, 107.0)
- added H3: MountingHole, MountingHole:MountingHole_3.2mm_M3, F.Cu at (114.0, 107.0)
- added H4: MountingHole, MountingHole:MountingHole_3.2mm_M3, F.Cu at (114.0, 61.0)
- added H5: MountingHole, MountingHole:MountingHole_3.2mm_M3, F.Cu at (169.0, 61.0)
- added R1: R, Resistor_THT:R_Axial_DIN0204_L3.6mm_D1.6mm_P7.62mm_Horizontal, F.Cu at (129.5, 67.5)
- moved H1 3.00 mm to (121.0, 98.0)
- moved PMOS1 3.00 mm to (125.0, 87.9)
Connections:
- PMOS1 pad 2: Net-(J1-Pad3) -> Net-(J2-Pad1)
- PMOS1 pad 3: Net-(J2-Pad1) -> Net-(J1-Pad3)
Routing:
- net Net-(J1-Pad2): track 121.7 -> 52.2 mm
- net Net-(J1-Pad3): track 61.7 -> 26.7 mm
- net Net-(J2-Pad1): track 33.8 -> 37.9 mm
