File: Motor Nucleo/MotorNucleo/MotorNucleo.kicad_pcb (KiCad board)
At the start: 2 copper layers, 71.1 x 57.2 mm, 11 parts, among them J1 Screw_Terminal_01x03, J10 Screw_Terminal_01x04, J11 Screw_Terminal_01x04, J2 Screw_Terminal_01x03, J3 Screw_Terminal_01x04, J4 Screw_Terminal_01x04, J5 Conn_01x15_Female, J6 Screw_Terminal_01x02, J7 Conn_01x15_Female, J8 Conn_01x06_Female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

Commit message: Uploaded PCB for Motor Nucleo breakout board
Parts:
- removed J10, J11: Screw_Terminal_01x04, Connector_PinSocket_2.54mm:PinSocket_1x04_P2.54mm_Vertical
- removed J8, J9: Conn_01x06_Female, Connector_PinSocket_2.54mm:PinSocket_1x06_P2.54mm_Vertical
- added G***: LOGO, SCR LOGO:robot-image, F.Cu at (132.1, 86.4)
- added G***: LOGO, SCR LOGO:crab-image, F.Cu at (180.3, 86.4)
- added G***: LOGO, SCR LOGO:small-scr-logo, F.Cu at (172.7, 58.4)
- added N1: Nucleo-L432KC, Module:Arduino_Nano, F.Cu at (138.1, 80.5)
- added REF**: MountingHole_3.2mm_M3, MountingHole:MountingHole_3.2mm_M3, F.Cu at (130.8, 104.1)
- added REF**: MountingHole_3.2mm_M3, MountingHole:MountingHole_3.2mm_M3, F.Cu at (182.9, 104.1)
- added REF**: MountingHole_3.2mm_M3, MountingHole:MountingHole_3.2mm_M3, F.Cu at (182.9, 55.9)
- added REF**: MountingHole_3.2mm_M3, MountingHole:MountingHole_3.2mm_M3, F.Cu at (130.8, 55.9)
- J1: value Screw_Terminal_01x03 -> JST_01x02; footprint Connector_PinSocket_2.54mm:PinSocket_1x03_P2.54mm_Vertical -> Connector_JST:JST_EH_B2B-EH-A_1x02_P2.50mm_Vertical
- J2: value Screw_Terminal_01x03 -> JST_01x04; footprint Connector_PinSocket_2.54mm:PinSocket_1x03_P2.54mm_Vertical -> Connector_JST:JST_EH_B4B-EH-A_1x04_P2.50mm_Vertical
- J3: value Screw_Terminal_01x04 -> JST_01x04; footprint Connector_PinSocket_2.54mm:PinSocket_1x04_P2.54mm_Vertical -> Connector_JST:JST_EH_B4B-EH-A_1x04_P2.50mm_Vertical
- J4: value Screw_Terminal_01x04 -> JST_01x03; footprint Connector_PinSocket_2.54mm:PinSocket_1x04_P2.54mm_Vertical -> Connector_JST:JST_EH_B3B-EH-A_1x03_P2.50mm_Vertical
- J5: value Conn_01x15_Female -> JST_01x04; footprint Connector_PinSocket_2.54mm:PinSocket_1x15_P2.54mm_Vertical -> Connector_JST:JST_EH_B4B-EH-A_1x04_P2.50mm_Vertical
- J6: value Screw_Terminal_01x02 -> JST_01x04; footprint Connector_PinSocket_2.54mm:PinSocket_1x02_P2.54mm_Vertical -> Connector_JST:JST_EH_B4B-EH-A_1x04_P2.50mm_Vertical
- J7: value Conn_01x15_Female -> JST_01x03; footprint Connector_PinSocket_2.54mm:PinSocket_1x15_P2.54mm_Vertical -> Connector_JST:JST_EH_B3B-EH-A_1x03_P2.50mm_Vertical
- moved J1 252.2 mm to (141.0, 55.9), turned to 180 degrees
- moved J2 217.1 mm to (133.3, 95.5), turned to 0 degrees
- moved J7 214.1 mm to (163.8, 55.9), turned to 180 degrees
- moved J4 212.5 mm to (152.4, 55.9), turned to 180 degrees
- moved J3 196.5 mm to (147.3, 95.2)
- moved J5 172.9 mm to (161.3, 95.2)
- moved J6 163.9 mm to (175.3, 95.2), turned to 0 degrees
Connections:
- J1 pad 1: Net-(J1-Pad1) -> GND
- J1 pad 2: Net-(J1-Pad1) -> +5V
- J2 pad 1: Net-(J2-Pad1) -> LEFT_EN_A
- J2 pad 2: Net-(J2-Pad1) -> LEFT_EN_A
- J2 pad 3: GND -> LEFT_EN_B
- J3 pad 1: Net-(J3-Pad1) -> RIGHT_EN_A
- J3 pad 2: Net-(J3-Pad2) -> RIGHT_EN_A
- J3 pad 3: Net-(J3-Pad1) -> RIGHT_EN_B
- J3 pad 4: Net-(J3-Pad2) -> RIGHT_EN_B
- J4 pad 1: Net-(J4-Pad1) -> RIGHT_PWM
- J4 pad 2: Net-(J4-Pad2) -> RIGHT_PWM
- J4 pad 3: Net-(J4-Pad1) -> GND
- J5 pad 1: Net-(J5-Pad1) -> +5V
- J5 pad 2: Net-(J5-Pad2) -> ENCODER_LEFT_A
- J5 pad 3: Net-(J5-Pad3) -> ENCODER_LEFT_B
- J5 pad 4: Net-(J5-Pad4) -> GND
- J6 pad 1: GND -> +5V
- J6 pad 2: +12V -> ENCODER_RIGHT_A
- J7 pad 1: +12V -> LEFT_PWM
- J7 pad 2: GND -> LEFT_PWM
- J7 pad 3: Net-(J7-Pad3) -> GND
Routing:
- net GND: track 0.00 -> 98.9 mm
- net +5V: track 0.00 -> 78.9 mm
- net LEFT_EN_A: track 0.00 -> 23.7 mm
- net LEFT_EN_B: track 0.00 -> 22.7 mm
- net RIGHT_EN_A: track 0.00 -> 19.8 mm
- net RIGHT_EN_B: track 0.00 -> 19.8 mm
- net ENCODER_RIGHT_A: track 0.00 -> 17.6 mm
- net ENCODER_RIGHT_B: track 0.00 -> 17.6 mm
- net RIGHT_PWM: track 0.00 -> 15.9 mm
- net ENCODER_LEFT_B: track 0.00 -> 15.7 mm
- net ENCODER_LEFT_A: track 0.00 -> 15.7 mm
- net LEFT_PWM: track 0.00 -> 12.0 mm
- removed copper zone on B.Cu, net GND
Other:
- board outline removed
- board text added: "Designed by: Tyler Julian"
- board text added: "Sooner Competitive Robotics"
